File: hardware/inktime.sch (EAGLE design)
At the start: 105 parts, among them IC1 BQ25180YBGR, IC2 DRV2605YZFR, IC3 BMA423, IC9 RT6160AWSC, J1 503480-2400, J2 TC2030-IDC, J4 KH-TYPE-C-16P, Q1 20V/4.2A/52mΩ/1.4W, Q3 SI1308EDL-T1-GE3, U1 NRF52840_QF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

Commit message: Minor changes to schematic and PCB
Signed-off-by: XXMA16 <xxma1610@gmail.com>
Parts:
- C15: value 1.0uF -> 1uF
- C23, C27, C34, C42: value 0.1uF -> 100nF
- C43: value 4.7F -> 4.7uF
Connections:
- removed net D+: D3.I/O2_2, U1.D+@AD6
- removed net D-: D3.I/O1_2, U1.D-@AD4
- new net D_N: D3.I/O2_2, U1.D-@AD4
- new net D_P: D3.I/O1_2, U1.D+@AD6
Other:
- note added: "Buttons"
- note added: "DC/DC"
- note added: "E-Paper Display Connector"
- note added: "E-Paper Drive Circuit"
- note added: "Fuel Gauge"
- note added: "Haptic Driver"
- note added: "IMU"
- note added: "LiPo Charger"
- note added: "SWD"
- note added: "USB C Connector & ESD Protection"
- moved on the sheet: C1-EP-DR, C2-EP-DR, D2, D4, D5, J4, L5, Q3, R1_EP_DR, R1_USB, R2_EP_DR, R2_USB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
